Commit message: Desired state now visualized using stl + using quaternion for desired orn

File: lobster_simulator/data/scout-alpha-visual.urdf (robot description, URDF)
Before this commit: robot Model_URDF.SLDASM, 1 links, 0 joints
Links:
- link base_link: mass 54.954 -> 0; geometry visual mesh filename=./base_link.STL
